File: AS5600_Mockup/AS5600_Mockup.kicad_pcb (KiCad board)
At the start: 2 copper layers, 23 x 23 mm, 7 parts

Commit message: Random changes
Parts:
- moved REF** 0.71 mm to (-8.00, 8.00)
- moved REF** 0.71 mm to (8.00, 8.00)
- moved REF** 0.71 mm to (8.00, -8.00)
- moved REF** 0.71 mm to (-8.00, -8.00)
Changed lines of the file:
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@@
 	(footprint "MountingHole:MountingHole_3.5mm"
 		(layer "F.Cu")
-		(at 8.5 8.5)
+		(at 8 8)
 		(descr "Mounting Hole 3.5mm, no annular, generated by kicad-footprint-generator mountinghole.py")
 		(tags "mountinghole")
@@
 	(footprint "MountingHole:MountingHole_3.5mm"
 		(layer "F.Cu")
-		(at -8.499999 8.499999)
+		(at -7.999999 7.999999)
 		(descr "Mounting Hole 3.5mm, no annular, generated by kicad-footprint-generator mountinghole.py")
 		(tags "mountinghole")
@@
 	(footprint "MountingHole:MountingHole_3.5mm"
 		(layer "F.Cu")
-		(at 8.5 -8.5)
+		(at 8 -8)
 		(descr "Mounting Hole 3.5mm, no annular, generated by kicad-footprint-generator mountinghole.py")
 		(tags "mountinghole")
@@
 	(footprint "MountingHole:MountingHole_3.5mm"
 		(layer "F.Cu")
-		(at -8.5 -8.5)
+		(at -8 -8)
 		(descr "Mounting Hole 3.5mm, no annular, generated by kicad-footprint-generator mountinghole.py")
 		(tags "mountinghole")
