File: Hydra_Driver/Driver_Unit.kicad_sch (KiCad schematic)
At the start: 21 parts, among them IC2 DRV8313RHHR, U3 INA199xxDCK, U4 INA199xxDCK

Commit message: Finished routing for Hydra V2
Parts:
- removed C17, C18, C20, C21: 0.1u, Capacitor_SMD:C_0402_1005Metric, symbol Device:C_Small
- removed R11, R15: 25m, Resistor_SMD:R_0603_1608Metric, symbol Device:R
- removed U3, U4: INA199xxDCK, Package_TO_SOT_SMD:SOT-363_SC-70-6, symbol Amplifier_Current:INA199xxDCK
- added C203, C204, C205: 1n, Capacitor_SMD:C_0402_1005Metric, symbol Device:C_Small
- added C208: 0.1u, Capacitor_SMD:C_0402_1005Metric, symbol Device:C_Small
- added R201, R202, R203, R204, R205, R206: 47, Resistor_SMD:R_0402_1005Metric, symbol Device:R
- added R212, R213, R214: 25m, Resistor_SMD:R_1206_3216Metric, symbol Device:R
- added U201: INA4181A2IPWR, Touchstone:PW20_TEX, symbol INA4181A2IPWR:INA4181A2IPWR
- renumbered C13 to C201, C14 to C202, C15 to C206, C16 to C207, C19 to C209, C22 to C210, D4 to D201, IC2 to IC201, R12 to R207, R13 to R208, R14 to R209, R16 to R210, R17 to R211
Connections:
- net +3.3V: now also C208.2, U201.5 (VS)
- net GND: now also C208.1, R202.2, R204.2, R206.2, R212.2, R213.2, R214.2, U201.1 (REF1), U201.12 (REF3), U201.16 (GND), U201.9 (REF2); no longer IC201.16 (PGND3)
- net SENSE1: now also U201.2 (OUT1)
- net SENSE2: now also U201.8 (OUT2)
- net SGND1: now also R201.2, R212.1
- net SGND2: now also R203.2, R213.1
- new net IN+1: C203.2, R201.1, U201.4 (IN+1)
- new net IN+2: C204.2, R203.1, U201.6 (IN+2)
- new net IN+3: C205.2, R205.1, U201.15 (IN+3)
- new net IN-1: C203.1, R202.1, U201.3 (IN-1)
- new net IN-2: C204.1, R204.1, U201.7 (IN-2)
- new net IN-3: C205.1, R206.1, U201.14 (IN-3)
- new net SENSE3: U201.13 (OUT3)
- new net SGND3: IC201.16 (PGND3), R205.2, R214.1
- no-connect marks 0 -> 4
Other:
- moved on the sheet: D201, R211
