File: Hydra_Driver/Driver_Unit.kicad_sch (KiCad schematic)
At the start: 27 parts, among them IC201 DRV8313RHHR, U201 INA4181A2IPWR

Commit message: Fixed SPI daisy chain issue
Parts:
- IC201: footprint Touchstone:QFN50P600X600X100-37N-D -> Touchscape:QFN50P600X600X100-37N-D
- U201: footprint Touchstone:PW20_TEX -> Touchscape:PW20_TEX
Changed lines of the file:
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@@
 			)
 		)
-		(property "Footprint" "Touchstone:PW20_TEX"
+		(property "Footprint" "Touchscape:PW20_TEX"
 			(at 96.52 140.97 0)
 			(effects
@@
 			)
 		)
-		(property "Footprint" "Touchstone:QFN50P600X600X100-37N-D"
+		(property "Footprint" "Touchscape:QFN50P600X600X100-37N-D"
 			(at 110.49 135.56 0)
 			(effects

Commit message: Fixed Kelvin connections and filter circuits
Parts:
- C203, C204, C205: value 1n -> 22n
- R201, R202, R203, R204, R205, R206: value 47 -> 10
- U201: value INA4181A2IPWR -> INA4181A3IPWR
Changed lines of the file:
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@@
 			)
 		)
-		(property "Value" "47"
+		(property "Value" "10"
 			(at 59.69 129.54 90)
 			(effects
@@
 			)
 		)
-		(property "Value" "1n"
+		(property "Value" "22n"
 			(at 68.58 172.7135 0)
 			(effects
@@
 			)
 		)
-		(property "Value" "47"
+		(property "Value" "10"
 			(at 59.69 172.72 90)
 			(effects
@@
 			)
 		)
-		(property "Value" "INA4181A2IPWR"
+		(property "Value" "INA4181A3IPWR"
 			(at 116.84 133.35 0)
 			(effects
@@
 			)
 		)
-		(property "Value" "47"
+		(property "Value" "10"
 			(at 59.69 162.56 90)
 			(effects
@@
 			)
 		)
-		(property "Value" "1n"
+		(property "Value" "22n"
 			(at 68.58 151.1235 0)
 			(effects
@@
 			)
 		)
-		(property "Value" "47"
+		(property "Value" "10"
 			(at 59.69 140.97 90)
 			(effects
@@
 			)
 		)
-		(property "Value" "47"
+		(property "Value" "10"
 			(at 59.69 119.38 90)
 			(effects
@@
 			)
 		)
-		(property "Value" "47"
+		(property "Value" "10"
 			(at 59.69 151.13 90)
 			(effects
@@
 			)
 		)
-		(property "Value" "1n"
+		(property "Value" "22n"
 			(at 68.58 129.5335 0)
 			(effects
