File: Hydra_Driver/Hydra_Driver.kicad_pcb (KiCad board)
At the start: 2 copper layers, 59.2 x 42 mm, 88 parts, among them IC1 ESP32-S3-WROOM-1-N4, IC2 DRV8313RHHR, IC3 DRV8313RHHR, J1 USB4105-GF-A, J10 Conn_01x03, J11 Conn_01x04, J12 Conn_01x03, J13 Conn_01x02, J2 Conn_01x02, J3 Conn_01x06, J4 Conn_01x03, J5 Conn_01x04, J6 Conn_01x03, J7 Conn_01x02, J8 Conn_01x03, J9 Conn_01x06, SW1 SW_SPST, SW2 SW_SPST, U1 USBLC6-2SC6, U2 MIC5504-3.3YM5-TR, U3 INA199xxDCK, U4 INA199xxDCK, U5 INA199xxDCK, U6 INA199xxDCK

Commit message: Finished routing for Hydra V2
Parts:
- removed C11, C17, C18, C20, C21, C27, C28, C30, C31, C9: 0.1u, Capacitor_SMD:C_0402_1005Metric
- removed J10, J4, J8: Conn_01x03, Connector_PinSocket_2.54mm:PinSocket_1x03_P2.54mm_Vertical
- removed J7: Conn_01x02, Connector_PinHeader_2.54mm:PinHeader_1x02_P2.54mm_Vertical
- removed R11, R15, R18, R22: 25m, Resistor_SMD:R_0603_1608Metric
- removed R8: 10k, Resistor_SMD:R_0402_1005Metric
- removed the REF** at (39.4, 39.4)
- removed the REF** at (50.2, 10.0)
- removed the REF** at (2.60, 30.0)
- removed U3, U4, U5, U6: INA199xxDCK, Package_TO_SOT_SMD:SOT-363_SC-70-6
- added C109: 0.1u, Capacitor_SMD:C_0402_1005Metric, F.Cu at (36.9, 1.97)
- added C111: 0.1u, Capacitor_SMD:C_0402_1005Metric, F.Cu at (26.7, 2.00)
- added C113: 0.1u, Capacitor_SMD:C_0402_1005Metric, F.Cu at (26.5, 41.0)
- added C203: 1n, Capacitor_SMD:C_0402_1005Metric, F.Cu at (54.8, 40.2)
- added C204: 1n, Capacitor_SMD:C_0402_1005Metric, F.Cu at (54.8, 36.0)
- added C205: 1n, Capacitor_SMD:C_0402_1005Metric, F.Cu at (54.8, 32.0)
- added C208: 0.1u, Capacitor_SMD:C_0402_1005Metric, F.Cu at (37.8, 36.2)
- added C303: 1n, Capacitor_SMD:C_0402_1005Metric, F.Cu at (54.8, 26.8)
- added C304: 1n, Capacitor_SMD:C_0402_1005Metric, F.Cu at (54.7, 22.5)
- added C305: 1n, Capacitor_SMD:C_0402_1005Metric, F.Cu at (54.8, 18.2)
- added C308: 0.1u, Capacitor_SMD:C_0402_1005Metric, F.Cu at (47.4, 5.73)
- added R201: 47, Resistor_SMD:R_0402_1005Metric, F.Cu at (52.6, 40.2)
- added R202: 47, Resistor_SMD:R_0402_1005Metric, F.Cu at (56.8, 40.2)
- added R203: 47, Resistor_SMD:R_0402_1005Metric, F.Cu at (52.6, 36.0)
- added R204: 47, Resistor_SMD:R_0402_1005Metric, F.Cu at (56.8, 36.0)
- added R205: 47, Resistor_SMD:R_0402_1005Metric, F.Cu at (52.6, 32.0)
- added R206: 47, Resistor_SMD:R_0402_1005Metric, F.Cu at (56.8, 32.0)
- added R212: 25m, Resistor_SMD:R_1206_3216Metric, F.Cu at (54.0, 38.2)
- added R213: 25m, Resistor_SMD:R_1206_3216Metric, F.Cu at (54.0, 34.0)
- added R214: 25m, Resistor_SMD:R_1206_3216Metric, F.Cu at (54.0, 30.0)
- added R301: 47, Resistor_SMD:R_0402_1005Metric, F.Cu at (52.6, 26.8)
- added R302: 47, Resistor_SMD:R_0402_1005Metric, F.Cu at (56.8, 26.8)
- added R303: 47, Resistor_SMD:R_0402_1005Metric, F.Cu at (52.6, 22.5)
- added R304: 47, Resistor_SMD:R_0402_1005Metric, F.Cu at (56.8, 22.5)
- added R305: 47, Resistor_SMD:R_0402_1005Metric, F.Cu at (52.6, 18.2)
- added R306: 47, Resistor_SMD:R_0402_1005Metric, F.Cu at (56.8, 18.2)
- added R312: 25m, Resistor_SMD:R_1206_3216Metric, F.Cu at (54.0, 24.8)
- added R313: 25m, Resistor_SMD:R_1206_3216Metric, F.Cu at (54.0, 20.5)
- added R314: 25m, Resistor_SMD:R_1206_3216Metric, F.Cu at (54.0, 16.5)
- added REF**: MountingHole_2.2mm_M2, MountingHole:MountingHole_2.2mm_M2, F.Cu at (49.2, 2.75)
- added REF**: MountingHole_2.2mm_M2, MountingHole:MountingHole_2.2mm_M2, F.Cu at (40.0, 39.2)
- added REF**: MountingHole_2.2mm_M2, MountingHole:MountingHole_2.2mm_M2, F.Cu at (4.00, 9.75)
- added REF**: MountingHole_2.2mm_M2, MountingHole:MountingHole_2.2mm_M2, F.Cu at (4.00, 32.2)
- added U103: SN74LVC1G373DCKR, Touchstone:SOT65P210X110-6N, F.Cu at (26.0, 38.5)
- added U201: INA4181A2IPWR, Touchstone:PW20_TEX, F.Cu at (33.2, 36.8)
- added U301: INA4181A2IPWR, Touchstone:PW20_TEX, F.Cu at (42.2, 4.25)
- J102: renamed from J2; footprint TerminalBlock:TerminalBlock_MaiXu_MX126-5.0-02P_1x02_P5.00mm -> Touchstone:AMASS_XT30U-F_1x02_P5.0mm_Vertical
- J104: renamed from J5; footprint Connector_PinHeader_2.54mm:PinHeader_1x04_P2.54mm_Horizontal -> Touchstone:CONN_CCSH-W10R-04TR-BK-A_ADA; moved to F.Cu
- J105: renamed from J6; footprint Connector_PinHeader_2.54mm:PinHeader_1x03_P2.54mm_Horizontal -> Connector_JST:JST_XH_S3B-XH-A-1_1x03_P2.50mm_Horizontal
- J107: renamed from J11; footprint Connector_PinHeader_2.54mm:PinHeader_1x04_P2.54mm_Horizontal -> Touchstone:CONN_CCSH-W10R-04TR-BK-A_ADA; moved to F.Cu
- J108: renamed from J12; footprint Connector_PinHeader_2.54mm:PinHeader_1x03_P2.54mm_Horizontal -> Connector_JST:JST_XH_S3B-XH-A-1_1x03_P2.50mm_Horizontal
- J109: renamed from J13; footprint TerminalBlock:TerminalBlock_MaiXu_MX126-5.0-02P_1x02_P5.00mm -> Touchstone:AMASS_XT30U-F_1x02_P5.0mm_Vertical
- SW101: renamed from SW1; footprint Button_Switch_THT:SW_PUSH_6mm -> Touchstone:SW_B3U-1000P
- SW102: renamed from SW2; footprint Button_Switch_THT:SW_PUSH_6mm -> Touchstone:SW_B3U-1000P
- moved R107 22.2 mm to (20.2, 39.0)
- moved C107 20.4 mm to (20.2, 3.25), turned to -90 degrees
- moved R106 18.9 mm to (21.5, 3.25), turned to 90 degrees
- moved C110 16.7 mm to (21.5, 39.0)
- moved C112 14.9 mm to (28.4, 2.00)
- moved C108 14.9 mm to (35.2, 2.00)
- moved U102 14.9 mm to (31.8, 2.25)
- moved SW101 13.8 mm to (17.0, 3.25)
- moved SW102 13.7 mm to (17.0, 39.0), turned to 0 degrees
- moved J108 13.6 mm to (50.2, 17.8), turned to -90 degrees
- moved J107 10.1 mm to (55.0, 11.2), turned to 90 degrees
- moved J105 9.74 mm to (50.2, 31.2), turned to -90 degrees
- moved D102 9.64 mm to (33.9, 5.25)
- moved D103 9.64 mm to (33.9, 7.25)
- moved R108 9.64 mm to (36.4, 5.25)
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- renumbered C1 to C101, C2 to C102, C3 to C103, C4 to C104, C5 to C105, C6 to C106, C7 to C107, C8 to C108, C10 to C110, C12 to C112, C13 to C201, C14 to C202, C15 to C206, C16 to C207, C19 to C209, C22 to C210, C23 to C301, C24 to C302, C25 to C306, C26 to C307, C29 to C309, C32 to C310, D1 to D101, D2 to D102, D3 to D103, D4 to D201, D5 to D301, IC1 to IC101, IC2 to IC201, IC3 to IC301, J1 to J101, J3 to J103, J9 to J106, R1 to R101, R2 to R102, R3 to R103, R4 to R104, R5 to R105, R6 to R106, R7 to R107, R9 to R108, R10 to R109, R12 to R207, R13 to R208, R14 to R209, R16 to R210, R17 to R211, R19 to R307, R20 to R308, R21 to R309, R23 to R310, R24 to R311, U1 to U101, U2 to U102
Connections:
- IC101 pad 10: /SENSE1A -> /SENSE2A
- IC101 pad 11: /IN1A -> /SENSE1A
- IC101 pad 12: unconnected-(IC1-IO8-Pad12) -> /IN1A
- IC101 pad 5: unconnected-(IC1-IO5-Pad5) -> /SENSE3B
- IC101 pad 8: /CS -> /CSIN
- IC101 pad 9: /SENSE2A -> /SENSE3A
- IC201 pad 16: GND -> /Driver_Unit/SGND3
- IC301 pad 16: GND -> /Driver_Unit1/SGND3
- J103 pad 1: /CS -> /CSCK
- J103 pad 2: /CLK -> /CSIN
- J103 pad 3: /LOOP1 -> /CLK
- J105 pad 1: /OUT1A -> /OUT3A
- J105 pad 3: /OUT3A -> /OUT1A
- J106 pad 1: /CS -> /CSCK
- J106 pad 2: /CLK -> /CSOUT
- J106 pad 3: /LOOP2 -> /CLK
- J108 pad 1: /OUT1B -> /OUT3B
- J108 pad 3: /OUT3B -> /OUT1B
Routing:
- net +3.3V: track 158.4 -> 217.9 mm, vias 10 -> 8
- net /CSOUT: track 0.00 -> 51.2 mm, vias 0 -> 1
- net /SENSE3B: track 0.00 -> 46.8 mm
- net /CSCK: track 0.00 -> 45.7 mm
- net /LOOP1: track 45.5 -> 0.00 mm
- net /CS: track 43.8 -> 0.00 mm, vias 3 -> 0
- net VMOT: track 136.6 -> 177.6 mm
- net /SENSE2A: track 44.1 -> 8.46 mm
- net /Driver_Unit/IN-3: track 0.00 -> 30.9 mm, vias 0 -> 2
- net /Driver_Unit/IN+3: track 0.00 -> 30.8 mm, vias 0 -> 2
- net /Driver_Unit/IN-2: track 0.00 -> 27.5 mm, vias 0 -> 2
- net /Driver_Unit1/IN+1: track 0.00 -> 27.0 mm, vias 0 -> 2
- net /Driver_Unit1/IN-1: track 0.00 -> 26.5 mm, vias 0 -> 2
- net /Driver_Unit1/IN-2: track 0.00 -> 25.4 mm, vias 0 -> 2
- net /Driver_Unit1/IN+2: track 0.00 -> 24.4 mm, vias 0 -> 2
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Other:
- board size 59.2 x 42 mm -> 58 x 42 mm
- board text removed: "+5V"
- board text removed: "1.0"
- board text removed: "BOOT"
- board text removed: "CLK"
- board text removed: "CS"
- board text removed: "HYDRA"
- board text removed: "I2C2"
- board text removed: "L1"
- board text removed: "L2"
- board text removed: "LED"
- board text removed: "MISO"
- board text removed: "MOSI"
- board text removed: "MTRA"
- board text removed: "MTRB"
- board text removed: "NSHIELD"
- board text removed: "PWR"
- board text removed: "SCL"
- board text removed: "SDA"
- board text removed: "VMOT"
- board text removed: "©CGR"

Commit message: Used correct flip flop for CS sequencing, added pullup
Parts:
- added R110: 10k, Resistor_SMD:R_0402_1005Metric, F.Cu at (28.0, 32.5)
- U103: value SN74LVC1G373DCKR -> SN74LVC1G80DBVR; footprint Touchstone:SOT65P210X110-6N -> Touchstone:DBV5
- moved C113 2.00 mm to (24.5, 41.0)
- moved U103 0.75 mm to (25.2, 38.5), turned to 180 degrees
Connections:
- IC101 pad 8: /CSIN -> /CSOUT
- U103 pad 1: /CSCK -> /CSIN
- U103 pad 2: GND -> /CSCK
- U103 pad 3: /CSIN -> GND
Routing:
- net /CSIN: track 10.5 -> 5.74 mm, vias 1 -> 0
- net /CSCK: track 45.7 -> 48.0 mm
- net +3.3V: track 217.9 -> 219.1 mm
- net /CSOUT: track 51.2 -> 51.6 mm, vias 1 -> 2
