File: Hydra_Driver/Hydra_Driver.kicad_sch (KiCad schematic)
At the start: 41 parts, among them IC101 ESP32-S3-WROOM-1-N4, J101 USB4105-GF-A, J102 Conn_01x02, J103 Conn_01x06, J104 Conn_01x04, J105 Conn_01x03, J106 Conn_01x06, J107 Conn_01x04, J108 Conn_01x03, J109 Conn_01x02, SW101 SW_SPST, SW102 SW_SPST, U101 USBLC6-2SC6, U102 MIC5504-3.3YM5-TR, U103 SN74LVC1G80DBVR

Commit message: Fixed SPI daisy chain issue
Parts:
- removed J103: Conn_01x06, Connector_PinSocket_2.54mm:PinSocket_1x06_P2.54mm_Horizontal, symbol Connector_Generic:Conn_01x06
- removed J106: Conn_01x06, Connector_PinHeader_2.54mm:PinHeader_1x06_P2.54mm_Horizontal, symbol Connector_Generic:Conn_01x06
- added J103: Conn_01x07, Connector_PinSocket_2.54mm:PinSocket_1x07_P2.54mm_Horizontal, symbol Connector_Generic:Conn_01x07
- added J110: Conn_01x07, Connector_PinHeader_2.54mm:PinHeader_1x07_P2.54mm_Horizontal, symbol Connector_Generic:Conn_01x07
- IC101: footprint Touchstone:ESP32S3WROOM1N4 -> Touchscape:ESP32S3WROOM1N4
- J101: footprint Touchstone:GCT_USB4105-GF-A -> Touchscape:GCT_USB4105-GF-A
- J102, J109: footprint Touchstone:AMASS_XT30U-F_1x02_P5.0mm_Vertical -> Touchscape:AMASS_XT30U-F_1x02_P5.0mm_Vertical
- J104, J107: footprint Touchstone:CONN_CCSH-W10R-04TR-BK-A_ADA -> Touchscape:CONN_CCSH-W10R-04TR-BK-A_ADA
- SW101, SW102: footprint Touchstone:SW_B3U-1000P -> Touchscape:SW_B3U-1000P
- U102: footprint Touchstone:SOT-23-5_MC_MCH -> Touchscape:SOT-23-5_MC_MCH
- U103: footprint Touchstone:DBV5 -> Touchscape:DBV5
Connections:
- net +5V: now also J103.7 (Pin_7), J110.7 (Pin_7)
- net CLK: now also J103.3 (Pin_3), J110.3 (Pin_3)
- net CSCK: now also J103.1 (Pin_1), J110.1 (Pin_1)
- net CSIN: now also IC101.8 (IO15), R110.2, J103.2 (Pin_2)
- net CSOUT: now also J110.2 (Pin_2); no longer IC101.8 (IO15), R110.2
- net GND: now also J103.6 (Pin_6), J110.6 (Pin_6)
- net MISO: now also J103.4 (Pin_4), J110.4 (Pin_4)
- net MOSI: now also J103.5 (Pin_5), J110.5 (Pin_5)
Other:
- moved on the sheet: R110
