File: Hydra_Encoder/Hydra_Encoder.kicad_pcb (KiCad board)
At the start: 2 copper layers, 30 x 30 mm, 14 parts, among them IC101 AS5600-ASOT, J101 Conn_01x04

Commit message: Panelized microcoder board
Parts:
- J101: footprint Touchstone:CONN_CCSH-W10R-04TR-BK-A_ADA -> Touchscape:CONN_CCSH-W10R-04TR-BK-A_ADA
Changed lines of the file:
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@@
 		)
 	)
-	(footprint "Touchstone:CONN_CCSH-W10R-04TR-BK-A_ADA"
+	(footprint "Touchscape:CONN_CCSH-W10R-04TR-BK-A_ADA"
 		(layer "F.Cu")
 		(at 0 12)
@@
 		)
 		(embedded_fonts no)
-		(model "C:/Users/carso/Documents/GitHub/Project-Touchstone/Touchstone-PCB/models/JST-XS-1x4-H.step"
+		(model "C:/Users/carso/Documents/GitHub/Project-Touchscape/Touchscape-PCB/models/JST-XS-1x4-H.step"
 			(offset
 				(xyz 0 0 0)
