File: Hydra_Encoder/Hydra_Encoder.kicad_sch (KiCad schematic)
At the start: 10 parts, among them IC101 AS5600-ASOT, J101 Conn_01x04

Commit message: Panelized microcoder board
Parts:
- J101: footprint Touchstone:CONN_CCSH-W10R-04TR-BK-A_ADA -> Touchscape:CONN_CCSH-W10R-04TR-BK-A_ADA
Changed lines of the file:
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@@
 			)
 		)
-		(property "Footprint" "Touchstone:CONN_CCSH-W10R-04TR-BK-A_ADA"
+		(property "Footprint" "Touchscape:CONN_CCSH-W10R-04TR-BK-A_ADA"
 			(at 120.65 36.83 0)
 			(effects
