File: Microcoder/Microcoder.kicad_pcb (KiCad board)
At the start: 2 copper layers, 12 x 12 mm, 7 parts, among them IC101 AS5600-ASOT, J101 Conn_01x04

Commit message: Panelized microcoder board
Parts:
- J101: footprint Touchstone:CONN_CCSH-W10R-04TR-BK-A_ADA -> Touchscape:CONN_CCSH-W10R-04TR-BK-A_ADA
Changed lines of the file:
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@@
 			(outputformat 1)
 			(mirror no)
-			(drillshape 1)
+			(drillshape 0)
 			(scaleselection 1)
-			(outputdirectory "")
+			(outputdirectory "./fab")
 		)
 	)
@@
 		)
 		(sheetname "/")
-		(sheetfile "Encoder_Button.kicad_sch")
+		(sheetfile "Microcoder.kicad_sch")
 		(attr smd)
 		(fp_line
@@
 		)
 	)
-	(footprint "Touchstone:CONN_CCSH-W10R-04TR-BK-A_ADA"
+	(footprint "Touchscape:CONN_CCSH-W10R-04TR-BK-A_ADA"
 		(layer "F.Cu")
 		(at 0 6)
@@
 			(unlocked yes)
 			(layer "F.SilkS")
-			(hide yes)
 			(effects
 				(font
@@
 		(property ki_fp_filters "Connector*:*_1x??_*")
 		(sheetname "/")
-		(sheetfile "Encoder_Button.kicad_sch")
+		(sheetfile "Microcoder.kicad_sch")
 		(attr smd)
 		(fp_line
@@
 		)
 		(embedded_fonts no)
-		(model "C:/Users/carso/Documents/GitHub/Project-Touchstone/Touchstone-PCB/models/JST-XS-1x4-H.step"
+		(model "C:/Users/carso/Documents/GitHub/Project-Touchscape/Touchscape-PCB/models/JST-XS-1x4-H.step"
 			(offset
 				(xyz 0 0 0)
@@
 		(property ki_fp_filters "R_*")
 		(sheetname "/")
-		(sheetfile "Encoder_Button.kicad_sch")
+		(sheetfile "Microcoder.kicad_sch")
 		(attr smd)
 		(fp_line
@@
 		(property ki_fp_filters "C_*")
 		(sheetname "/")
-		(sheetfile "Encoder_Button.kicad_sch")
+		(sheetfile "Microcoder.kicad_sch")
 		(attr smd)
 		(fp_line
@@
 		(property ki_fp_filters "R_*")
 		(sheetname "/")
-		(sheetfile "Encoder_Button.kicad_sch")
+		(sheetfile "Microcoder.kicad_sch")
 		(attr smd)
 		(fp_line
@@
 		(property ki_fp_filters "R_*")
 		(sheetname "/")
-		(sheetfile "Encoder_Button.kicad_sch")
+		(sheetfile "Microcoder.kicad_sch")
 		(attr smd)
 		(fp_line
@@
 		(property ki_fp_filters "C_*")
 		(sheetname "/")
-		(sheetfile "Encoder_Button.kicad_sch")
+		(sheetfile "Microcoder.kicad_sch")
 		(attr smd)
 		(fp_line
